File: KiCad Project/ts_808.kicad_pcb (KiCad board)
At the start: 2 copper layers, 75 x 52 mm, 61 parts, among them Q1 2SC1815, Q2 2SC1815, U1 RC4558

Commit message: Full project commit
Other:
- board text added: "127.00 mm"
- board text added: "52.00 mm"
- board text added: "75.00 mm"
- board text added: "76.250 mm"
